Commit message: Add thruster links and joints to easys.urdf

File: Easys_description/model/urdf/easys.urdf (robot description, URDF)
Before this commit: robot test_robot, 2 links, 1 joints
Links:
- added link left_down_thruster_link; visual cylinder length=0.1 radius=0.05
- added link left_up_thruster_link; visual cylinder length=0.1 radius=0.05
- added link right_down_thruster_link; visual cylinder length=0.1 radius=0.05
- added link right_up_thruster_link; visual cylinder length=0.1 radius=0.05
Joints:
- added joint left_down_thruster_joint: type fixed, parent base_link, child left_down_thruster_link, origin xyz=0.2 0 0 rpy=0 0 -1.57
- added joint left_up_thruster_joint: type fixed, parent base_link, child left_up_thruster_link, origin xyz=0.5 0 0 rpy=0 0.785 0
- added joint right_down_thruster_joint: type fixed, parent base_link, child right_down_thruster_link, origin xyz=-0.2 0 0 rpy=0 0 -1.57
- added joint right_up_thruster_joint: type fixed, parent base_link, child right_up_thruster_link, origin xyz=-0.5 0 0 rpy=0 0.785 3.14

Commit message: update urdf

File: Easys_description/model/urdf/easys.urdf (robot description, URDF)
Before this commit: robot test_robot, 6 links, 5 joints
Links:
- link left_down_thruster_link: geometry 
- link left_up_thruster_link: geometry 
- link right_down_thruster_link: geometry 
- link right_up_thruster_link: geometry 
Joints:
- joint left_down_thruster_joint: origin xyz=0.2 0 0 rpy=0 0 -1.57 -> xyz=0.116 0.1145 0.1215 rpy=0 0 -1.57
- joint left_up_thruster_joint: origin xyz=0.5 0 0 rpy=0 0.785 0 -> xyz=0.08255 0 0.22255 rpy=0 0.785 0
- joint right_down_thruster_joint: origin xyz=-0.2 0 0 rpy=0 0 -1.57 -> xyz=-0.116 0 0.1215 rpy=0 0 -1.57
- joint right_up_thruster_joint: origin xyz=-0.5 0 0 rpy=0 0.785 3.14 -> xyz=-0.08255 0 0.22255 rpy=0 0.785 3.14

Commit message: urdf ok

File: Easys_description/model/urdf/easys.urdf (robot description, URDF)
Before this commit: robot test_robot, 6 links, 5 joints
Joints:
- joint left_down_thruster_joint: origin xyz=0.116 0.1145 0.1215 rpy=0 0 -1.57 -> xyz=0.116 0.04715 0.1215 rpy=0 0 -1.57
- joint right_down_thruster_joint: origin xyz=-0.116 0 0.1215 rpy=0 0 -1.57 -> xyz=-0.116 0.04715 0.1215 rpy=0 0 -1.57
